File: aab/aab.kicad_pcb (KiCad board)
At the start: 2 copper layers, 64 x 67.5 mm, 34 parts

Commit message: Update AAB pcb design
Parts:
- REF** (x2): value PinHeader_1x03_P2.54mm_Vertical -> PinHeader_1x03_P2.54mm_Horizontal; footprint Connector_PinHeader_2.54mm:PinHeader_1x03_P2.54mm_Vertical -> Connector_PinHeader_2.54mm:PinHeader_1x03_P2.54mm_Horizontal
- moved REF** 6.02 mm to (86.9, 142.0), turned to 180 degrees
- moved REF** 2.53 mm to (79.9, 85.6), turned to 0 degrees
Routing:
- net DOUT: track 7.78 -> 22.5 mm
- net DIN2: track 11.4 -> 15.9 mm
- net VSS: vias 12 -> 11
Other:
- board text added: "LUX - AAB - v2019.09.29"
- board text removed: "LUX - AAB - v2019.09.28"
