File: bcc/bcc.kicad_pcb (KiCad board)
At the start: 2 copper layers, 67.2 x 125.9 mm, 62 parts

Commit message: Update BCC PCB
Parts:
- removed the VSS at (50.0, 36.2)
- added VSS: BridgeSolderPad_3xinline, Dex connectors:BridgeSolderPad_3xinline, F.Cu at (50.0, 36.2)
- D1, D10, D11, D12, D13, D14, D15, D16, D17, D18, D19, D2, D20, D21, D22, D23, D24, D3, D4, D5, D6, D7, D8, D9: footprint SK6412_BIG_PAD -> Dex leds:SK6812_BIG_PAD
- REF** (x2): value PinHeader_1x03_P2.54mm_Vertical -> PinHeader_1x03_P2.54mm_Horizontal; footprint PinHeader_1x03_P2.54mm_Vertical -> Connector_PinHeader_2.54mm:PinHeader_1x03_P2.54mm_Horizontal
- REF** (x2), VDD (x2), VSS (x3): footprint BridgeSolderPad_3xinline -> Dex connectors:BridgeSolderPad_3xinline
- moved REF** 3.81 mm to (81.3, 142.0), turned to 180 degrees
- moved REF** 3.36 mm to (86.4, 27.2), turned to 0 degrees
- moved VSS 0.11 mm to (117.3, 138.1)
- turned C1 to 338.7 degrees
- turned C1 to 351.9 degrees
- turned C1 to 355 degrees
- turned C1 to 177.7 degrees
- turned C1 to 345.4 degrees
- turned C1 to 352.6 degrees
- turned C1 to 356.7 degrees
- turned C1 to 350.1 degrees
- turned C1 to 343.9 degrees
- turned C1 to 348.2 degrees
- turned C1 to 354 degrees
- turned C1 to 357.3 degrees
Routing:
- net VSS: track 113.5 -> 0.00 mm
- net VDD: track 115.9 -> 47.1 mm
- net DIN: track 14.9 -> 12.5 mm
- net Net-(D6-Pad4): track 29.5 -> 27.5 mm
- net D2: track 19.1 -> 17.3 mm
- net Net-(D10-Pad2): track 24.1 -> 22.8 mm
- net Net-(D1-Pad4): track 10.4 -> 11.6 mm
- net Net-(D13-Pad2): track 29.8 -> 28.6 mm
- net Net-(D22-Pad4): track 19.1 -> 19.9 mm
- net Net-(D4-Pad4): track 23.0 -> 22.1 mm
- net Net-(D23-Pad4): track 17.9 -> 17.2 mm
- net Net-(D18-Pad4): track 18.6 -> 19.3 mm
Other:
- board text added: "Designed in Italy with"
- board text added: "LUX - BCC - v2019.10.06"
- board text removed: "Designed in Italy with by"
- board text removed: "VDD x 2"
- board text removed: "v 2019.09.22"
